Commit message: Fix bugs

File: models/urdf/pipe.xacro (robot description, xacro)
@@ -11,5 +11,5 @@
   <xacro:property name="scale_t" value="${$(arg thickness)/50}" />
   <xacro:property name="pillar_length" value="${$(arg altitude)-0.1-$(arg radius)}" />
-  <xacro:property name="mesh_file" value="package://ss_workshop/models/meshes/Plain_Cylinder.stl" />
+  <xacro:property name="mesh_file" value="package://summer_school_world/models/meshes/Plain_Cylinder.stl" />
   <!-- Macro for the inertia of a box -->
   <xacro:macro name="box_inertia" params="x y z mass">
